Commit message: fix(descr): lidar gazebo frame fixed

File: waver_description/urdf/lidar.xacro (robot description, xacro)
@@ -3,5 +3,5 @@
     <xacro:include filename="$(find waver_description)/urdf/materials.xacro" />
     <xacro:include filename="$(find waver_description)/urdf/util.xacro" />
-    <link name="${lidar_link}">
+    <link name="lidar_link">
         <inertial>
             <mass value="${mass_lidar}" />
@@ -26,12 +26,13 @@
         <origin xyz="0.04 0 ${base_to_top + 0.025}" rpy="0 0 0" />
         <parent link="top_shell_link" />
-        <child link="${lidar_link}" />
+        <child link="lidar_link" />
     </joint>
-    <gazebo reference="${lidar_link}">
+    <gazebo reference="lidar_link">
         <material>Gazebo/Black</material>
-        <sensor name="${lidar_model}" type="gpu_lidar">
+        <sensor name="lidar_link" type="gpu_lidar">
             <pose>0 0 0 0 0 0</pose>
             <visualize>false</visualize>
             <topic>scan</topic>
+            <gz_frame_id>lidar_link</gz_frame_id>
             <always_on>true</always_on>
             <update_rate>${lidar_frequency}</update_rate>

File: waver_description/urdf/util.xacro (robot description, xacro)
@@ -92,6 +92,4 @@
     <!-- Lidar specifications -->
     <xacro:property name="mass_lidar" value="0.046" />
-    <xacro:property name="lidar_model" value="HLS-LFCD-LDS" />
-    <xacro:property name="lidar_link" value="lidar_link" />
     <xacro:property name="lidar_samples" value="720" />
     <xacro:property name="lidar_max_range" value="12.0" />
